File: hw/vwcdpic.kicad_pcb (KiCad board)
At the start: 2 copper layers, 14.6 x 13.1 mm, 12 parts, among them U1 PIC12F629, U2 LM78L05ACZ, U3 MC78L05ACH

Commit message: programing notes
Other:
- net class Default removed
- net class GND removed
- board text added: "PRG_DATA PRG_CLK GND"
- board text added: "RESET 5V"
