File: hw/vwcdpic.sch (KiCad schematic (older format))
At the start: 12 parts, among them U1 PIC12F629, U2 LM78L05ACZ, U3 MC78L05ACH

Commit message: update
Parts:
- C1: value 1uF/6.3V -> 1uF/16V; footprint Capacitors_Tantalum_SMD:TantalC_SizeA_EIA-3216_Reflow -> Capacitors_SMD:C_0805_HandSoldering
Changed lines of the file:
@@
 POWER_CTL
 $Comp
-L GND #PWR7
+L GND #PWR01
 U 1 1 52D3D3F9
 P 6900 3550
-F 0 "#PWR7" H 6900 3550 30  0001 C CNN
+F 0 "#PWR01" H 6900 3550 30  0001 C CNN
 F 1 "GND" H 6900 3480 30  0001 C CNN
 F 2 "" H 6900 3550 60  0001 C CNN
@@
 DataIn-PRG_CLK
 $Comp
-L +5V #PWR2
+L +5V #PWR02
 U 1 1 52D03030
 P 3400 2350
-F 0 "#PWR2" H 3400 2440 20  0001 C CNN
+F 0 "#PWR02" H 3400 2440 20  0001 C CNN
 F 1 "+5V" H 3400 2440 30  0000 C CNN
 F 2 "" H 3400 2350 60  0001 C CNN
@@
 $EndComp
 $Comp
-L +5V #PWR6
+L +5V #PWR03
 U 1 1 52D02FCA
 P 5950 5000
-F 0 "#PWR6" H 5950 5090 20  0001 C CNN
+F 0 "#PWR03" H 5950 5090 20  0001 C CNN
 F 1 "+5V" H 5950 5090 30  0000 C CNN
 F 2 "" H 5950 5000 60  0001 C CNN
@@
 $EndComp
 $Comp
-L GND #PWR3
+L GND #PWR04
 U 1 1 52D02FB7
 P 4850 3050
-F 0 "#PWR3" H 4850 3050 30  0001 C CNN
+F 0 "#PWR04" H 4850 3050 30  0001 C CNN
 F 1 "GND" H 4850 2980 30  0001 C CNN
 F 2 "" H 4850 3050 60  0001 C CNN
@@
 $EndComp
 $Comp
-L GND #PWR5
+L GND #PWR05
 U 1 1 52D02FA3
 P 5500 5950
-F 0 "#PWR5" H 5500 5950 30  0001 C CNN
+F 0 "#PWR05" H 5500 5950 30  0001 C CNN
 F 1 "GND" H 5500 5880 30  0001 C CNN
 F 2 "" H 5500 5950 60  0001 C CNN
@@
 $EndComp
 $Comp
-L GND #PWR4
+L GND #PWR06
 U 1 1 52D02FA1
 P 5050 5950
-F 0 "#PWR4" H 5050 5950 30  0001 C CNN
+F 0 "#PWR06" H 5050 5950 30  0001 C CNN
 F 1 "GND" H 5050 5880 30  0001 C CNN
 F 2 "" H 5050 5950 60  0001 C CNN
@@
 P 3150 4150
 F 0 "C1" H 3175 4250 50  0000 L CNN
-F 1 "1uF/6.3V" H 3175 4050 50  0000 L CNN
-F 2 "Capacitors_Tantalum_SMD:TantalC_SizeA_EIA-3216_Reflow" H 3188 4000 30  0000 C CNN
+F 1 "1uF/16V" H 3175 4050 50  0000 L CNN
+F 2 "Capacitors_SMD:C_0805_HandSoldering" H 3188 4000 30  0000 C CNN
 F 3 "" H 3150 4150 60  0000 C CNN
 	1    3150 4150
@@
 $EndComp
 $Comp
-L GND #PWR1
+L GND #PWR07
 U 1 1 55C4B8F3
 P 3150 4400
-F 0 "#PWR1" H 3150 4400 30  0001 C CNN
+F 0 "#PWR07" H 3150 4400 30  0001 C CNN
 F 1 "GND" H 3150 4330 30  0001 C CNN
 F 2 "" H 3150 4400 60  0001 C CNN
@@
 	7600 4300 7700 4300
 $Comp
-L +5V #PWR?
+L +5V #PWR08
 U 1 1 5617A229
 P 8000 5050
-F 0 "#PWR?" H 8000 5140 20  0001 C CNN
+F 0 "#PWR08" H 8000 5140 20  0001 C CNN
 F 1 "+5V" H 8000 5140 30  0000 C CNN
 F 2 "" H 8000 5050 60  0001 C CNN
@@
 POWER_CTL
 $Comp
-L GND #PWR?
+L GND #PWR09
 U 1 1 5617A2CE
 P 7400 5900
-F 0 "#PWR?" H 7400 5900 30  0001 C CNN
+F 0 "#PWR09" H 7400 5900 30  0001 C CNN
 F 1 "GND" H 7400 5830 30  0001 C CNN
 F 2 "" H 7400 5900 60  0001 C CNN

Commit message: hw upgrade
Parts:
- U3: footprint Housings_SOT-23_SOT-143_TSOT-6:SOT-23 -> TO_SOT_Packages_SMD:SOT-23_Handsoldering
Connections:
- net GND: now also U3.3 (IN); no longer U3.2 (GND)
- net POWER_CTL: now also U3.2 (GND); no longer U3.3 (IN)
Changed lines of the file:
@@
 F 0 "U3" H 7200 5450 40  0000 C CNN
 F 1 "MC78L05ACH" H 7400 5450 40  0000 L CNN
-F 2 "Housings_SOT-23_SOT-143_TSOT-6:SOT-23" H 7400 5350 30  0000 C CIN
+F 2 "TO_SOT_Packages_SMD:SOT-23_Handsoldering" H 7400 5350 30  0000 C CIN
 F 3 "" H 7400 5250 60  0000 C CNN
 	1    7400 5250
@@
 Wire Wire Line
 	8000 5050 8000 5200
-Wire Wire Line
-	8000 5200 7800 5200
-Wire Wire Line
-	7000 5200 6900 5200
-Wire Wire Line
-	7400 5900 7400 5500
 Wire Notes Line
 	6200 4900 8100 4900
@@
 Text Notes 6250 6000 0    60   ~ 0
 TO-23 78L05\nALTERNATIVE
+Wire Wire Line
+	7000 5200 7000 5800
+Wire Wire Line
+	7000 5800 7400 5800
+Wire Wire Line
+	7400 5800 7400 5900
+Wire Wire Line
+	7400 5500 7400 5550
+Wire Wire Line
+	7400 5550 6950 5550
+Wire Wire Line
+	6950 5550 6950 5200
+Wire Wire Line
+	6950 5200 6900 5200
+Wire Wire Line
+	8000 5200 7800 5200
 $EndSCHEMATC
