File: hw/vwcdpic_THT.kicad_pcb (KiCad board)
At the start: 2 copper layers, 31 x 16.6 mm, 11 parts, among them U1 PIC12F629, U2 LM78L05ACZ

Commit message: hw and pictures changes
Parts:
- U2: value LM78L05ACZ -> 78L05
Other:
- board text added: "+5V"
- board text added: "ARCHOS"
- board text added: "Acc"
- board text added: "CLK"
- board text added: "DataIN"
- board text added: "DataOut"
- board text added: "GND"
- board text added: "PJRC"
- board text added: "RESET"
Changed lines of the file:
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@@
-(kicad_pcb (version 4) (host pcbnew 0.201510080346+6253~30~ubuntu14.04.1-product)
+(kicad_pcb (version 20171130) (host pcbnew 5.0.0-rc3-unknown-3df2743~65~ubuntu16.04.1)
   (general
-    (links 22)
-    (no_connects 0)
-    (area 129.806699 127.022859 161.211261 143.974821)
     (thickness 1.6002)
-    (drawings 9)
+    (drawings 31)
     (tracks 76)
     (zones 0)
@@
     (pad_to_mask_clearance 0.254)
     (aux_axis_origin 0 0)
-    (visible_elements FFFEDBBF)
+    (visible_elements FFFEDBFF)
     (pcbplotparams
       (layerselection 0x0100f_80000001)
       (usegerberextensions false)
+      (usegerberattributes false)
+      (usegerberadvancedattributes false)
+      (creategerberjobfile false)
       (excludeedgelayer false)
       (linewidth 0.150000)
@@
       (hpglpennumber 1)
       (hpglpenspeed 20)
-      (hpglpendiameter 15)
-      (hpglpenoverlay 0)
+      (hpglpendiameter 15.000000)
       (psnegative false)
       (psa4output false)
@@
       (drillshape 0)
       (scaleselection 1)
-      (outputdirectory /home/nail/tmp/plot/))
+      (outputdirectory "/home/nail/tmp/plot/"))
   )
   (net 0 "")
@@
     (descr "Film Capacitor Length 7mm x Width 2.5mm, Pitch 5mm")
     (tags Capacitor)
-    (fp_text reference C3 (at 2.38252 -0.36576 270) (layer F.SilkS)
-      (effects (font (size 1 1) (thickness 0.15)))
-    )
-    (fp_text value 100n (at 2.5 2.5 270) (layer F.Fab)
+    (fp_text reference C3 (at 2.55524 -0.01016 270) (layer F.SilkS)
+      (effects (font (size 1 1) (thickness 0.15)))
+    )
+    (fp_text value 100n (at 5.06984 3.39344) (layer F.SilkS)
       (effects (font (size 1 1) (thickness 0.15)))
     )
@@
       (net 2 GND))
     (model Capacitors_ThroughHole.3dshapes/C_Disc_D6_P5.wrl
-      (at (xyz 0.1 0 0))
+      (offset (xyz 2.539999961853027 0 0))
       (scale (xyz 1 1 1))
       (rotate (xyz 0 0 0))
@@
       (effects (font (size 1 1) (thickness 0.15)))
     )
-    (fp_text value 100n (at 2.5 2.5 90) (layer F.Fab)
+    (fp_text value 100n (at -1.37668 2.2098) (layer F.SilkS)
       (effects (font (size 1 1) (thickness 0.15)))
     )
@@
       (net 2 GND))
     (model Capacitors_ThroughHole.3dshapes/C_Disc_D6_P5.wrl
-      (at (xyz 0.1 0 0))
+      (offset (xyz 2.539999961853027 0 0))
       (scale (xyz 1 1 1))
       (rotate (xyz 0 0 0))
@@
     (descr "Transistor TO92 brochage type BC237")
     (tags "TR TO92")
-    (fp_text reference U2 (at 0.021553 -3.038919 225) (layer F.SilkS)
-      (effects (font (size 1.016 1.016) (thickness 0.2032)))
-    )
-    (fp_text value LM78L05ACZ (at -1.27 -5.08 225) (layer F.SilkS) hide
-      (effects (font (size 1.016 1.016) (thickness 0.2032)))
+    (fp_text reference U2 (at -2.697669 -0.219118 225) (layer F.SilkS)
+      (effects (font (size 1 1) (thickness 0.15)))
+    )
+    (fp_text value 78L05 (at -0.021553 -2.895235 225) (layer F.SilkS)
+      (effects (font (size 1 1) (thickness 0.15)))
     )
     (fp_line (start -1.27 2.54) (end 2.54 -1.27) (layer F.SilkS) (width 0.3048))
@@
     (descr "8 pins DIL package, elliptical pads")
     (tags DIL)
-    (fp_text reference U1 (at 1.143 0.09652 360) (layer F.SilkS)
-      (effects (font (size 1 1) (thickness 0.15)))
-    )
-    (fp_text value PIC12F629 (at 0 0 270) (layer F.Fab)
+    (fp_text reference U1 (at 0.82296 -0.8382 90) (layer F.SilkS)
+      (effects (font (size 1 1) (thickness 0.15)))
+    )
+    (fp_text value PIC12F629 (at 0.77216 0.9398 270) (layer F.SilkS)
       (effects (font (size 1 1) (thickness 0.15)))
     )
@@
     (descr "Resistor, Axial,  RM 10mm, 1/3W,")
     (tags "Resistor, Axial, RM 10mm, 1/3W,")
-    (fp_text reference R7 (at 0.1016 0.0508) (layer F.SilkS)
-      (effects (font (size 1 1) (thickness 0.15)))
-    )
-    (fp_text value 3k3 (at 3.81 3.81) (layer F.Fab)
+    (fp_text reference R7 (at -1.53924 0.01016 90) (layer F.SilkS)
+      (effects (font (size 1 1) (thickness 0.15)))
+    )
+    (fp_text value 3k3 (at 0.74676 0.01016) (layer F.SilkS)
       (effects (font (size 1 1) (thickness 0.15)))
     )
@@
     (descr "Resistor, Axial,  RM 10mm, 1/3W,")
     (tags "Resistor, Axial, RM 10mm, 1/3W,")
-    (fp_text reference R6 (at 0.01524 -0.13208) (layer F.SilkS)
-      (effects (font (size 1 1) (thickness 0.15)))
-    )
-    (fp_text value 3k3 (at 3.81 3.81) (layer F.Fab)
+    (fp_text reference R6 (at -1.59004 0.0762 90) (layer F.SilkS)
+      (effects (font (size 1 1) (thickness 0.15)))
+    )
+    (fp_text value 3k3 (at 0.79756 0.0762) (layer F.SilkS)
       (effects (font (size 1 1) (thickness 0.15)))
     )
@@
     (descr "Resistor, Axial,  RM 10mm, 1/3W,")
     (tags "Resistor, Axial, RM 10mm, 1/3W,")
-    (fp_text reference R5 (at -0.0762 -0.0508) (layer F.SilkS)
-      (effects (font (size 1 1) (thickness 0.15)))
-    )
-    (fp_text value 3k3 (at 3.81 3.81) (layer F.Fab)
+    (fp_text reference R5 (at -1.59004 -0.01524 90) (layer F.SilkS)
+      (effects (font (size 1 1) (thickness 0.15)))
+    )
+    (fp_text value 3k3 (at 0.74676 0.16256) (layer F.SilkS)
       (effects (font (size 1 1) (thickness 0.15)))
     )
@@
     (descr "Radial Electrolytic Capacitor Diameter 5mm x Length 11mm, Pitch 2.5mm")
     (tags "Electrolytic Capacitor")
-    (fp_text reference C1 (at 2.39776 -3.6322 270) (layer F.SilkS)
-      (effects (font (size 1 1) (thickness 0.15)))
-    )
-    (fp_text value 1uF/6.3V (at 1.25 3.8 270) (layer F.Fab)
+    (fp_text reference C1 (at 1.57988 -3.92176) (layer F.SilkS)
+      (effects (font (size 1 1) (thickness 0.15)))
+    )
+    (fp_text value 1uF/6.3V (at 2.84988 -6.10616) (layer F.SilkS)
       (effects (font (size 1 1) (thickness 0.15)))
     )
@@
       (net 2 GND))
     (model Capacitors_ThroughHole.3dshapes/C_Radial_D5_L11_P2.5.wrl
-      (at (xyz 0.049213 0 0))
+      (offset (xyz 1.25001018122673 0 0))
       (scale (xyz 1 1 1))
       (rotate (xyz 0 0 90))
@@
     (descr "Resistor, Axial,  RM 10mm, 1/3W,")
     (tags "Resistor, Axial, RM 10mm, 1/3W,")
-    (fp_text reference R1 (at 0.06604 0.06096) (layer F.SilkS)
-      (effects (font (size 1 1) (thickness 0.15)))
-    )
-    (fp_text value 10k (at 3.81 3.81) (layer F.Fab)
+    (fp_text reference R1 (at -1.65608 -0.14224 90) (layer F.SilkS)
+      (effects (font (size 1 1) (thickness 0.15)))
+    )
+    (fp_text value 10k (at 0.78232 0.01016) (layer F.SilkS)
       (effects (font (size 1 1) (thickness 0.15)))
     )
@@
     )
   )
+  (gr_line (start 136.906 130.2766) (end 137.3886 129.9083) (layer B.SilkS) (width 0.1))
+  (gr_line (start 134.0612 130.2766) (end 136.906 130.2766) (layer B.SilkS) (width 0.1))
+  (gr_line (start 132.9563 129.3749) (end 134.0612 130.2766) (layer B.SilkS) (width 0.1))
+  (gr_line (start 137.2108 132.7277) (end 137.795 132.2578) (layer B.SilkS) (width 0.1))
+  (gr_line (start 134.2517 132.7404) (end 137.2108 132.7277) (layer B.SilkS) (width 0.1))
+  (gr_line (start 133.2103 131.9276) (end 134.2517 132.7404) (layer B.SilkS) (width 0.1))
+  (gr_line (start 137.4902 135.4201) (end 137.9093 134.9375) (layer B.SilkS) (width 0.1))
+  (gr_line (start 134.1882 135.4201) (end 137.4902 135.4201) (layer B.SilkS) (width 0.1))
+  (gr_line (start 133.0833 134.6581) (end 134.1882 135.4201) (layer B.SilkS) (width 0.1))
+  (gr_line (start 138.0363 137.414) (end 138.049 137.414) (layer B.SilkS) (width 0.1))
+  (gr_line (start 137.2743 137.922) (end 138.0363 137.414) (layer B.SilkS) (width 0.1))
+  (gr_line (start 134.2136 137.8839) (end 137.2743 137.922) (layer B.SilkS) (width 0.1))
+  (gr_line (start 133.2484 137.2362) (end 134.2136 137.8839) (layer B.SilkS) (width 0.1))
+  (gr_text +5V (at 139.446 136.7917) (layer B.SilkS)
+    (effects (font (size 1 1) (thickness 0.15)) (justify mirror))
+  )
+  (gr_text RESET (at 139.3825 134.1247) (layer B.SilkS)
+    (effects (font (size 1 0.8) (thickness 0.15)) (justify mirror))
+  )
+  (gr_text PJRC (at 139.319 131.699) (layer B.SilkS)
+    (effects (font (size 1 0.8) (thickness 0.15)) (justify mirror))
+  )
+  (gr_text ARCHOS (at 139.4968 129.1336) (layer B.SilkS)
+    (effects (font (size 1 0.8) (thickness 0.15)) (justify mirror))
+  )
+  (gr_text CLK (at 153.4668 128.8796) (layer B.SilkS)
+    (effects (font (size 1 1) (thickness 0.15)) (justify mirror))
+  )
+  (gr_text Acc (at 156.5529 139.1793) (layer B.SilkS)
+    (effects (font (size 1 1) (thickness 0.15)) (justify mirror))
+  )
+  (gr_text GND (at 154.3558 136.6266) (layer B.SilkS)
+    (effects (font (size 1 1) (thickness 0.15)) (justify mirror))
+  )
+  (gr_text "DataOut\n" (at 152.1079 134.1755) (layer B.SilkS)
+    (effects (font (size 1 1) (thickness 0.15)) (justify mirror))
+  )
+  (gr_text DataIN (at 152.4635 131.5974) (layer B.SilkS)
+    (effects (font (size 1 1) (thickness 0.15)) (justify mirror))
+  )
   (gr_line (start 129.9972 143.78432) (end 132.65912 143.78432) (angle 90) (layer Edge.Cuts) (width 0.381))
