File: hw/with_BT/vwcdpic_with_BT.kicad_pcb (KiCad board)
At the start: 2 copper layers, 68.1 x 49.8 mm, 102 parts, among them J1 Ant, J2 TMS, J3 TCK, J4 TDO, J5 TDI, J6 AUDIO, J7 3.5mmjack, J8 CDC, P1 7805, P2 ICSP, P3 AUX, P4 MIC_ALT, P5 SERIAL, Q1 BSS138, Q2 PMV65XPE, U1 AP1117-33, U3 TL072, U4 AP1117, U5 F-6988, U6 PIC12F629-ISN

Commit message: add (C)
Other:
- board text added: "(C) Tomas Kovacik vwcdpic + BK3266 v1"
Changed lines of the file:
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@@
+    (effects (font (size 0.8 0.8) (thickness 0.1)))
+  )
+  (gr_text "(C) Tomas Kovacik\nvwcdpic + BK3266\nv1" (at 100.9396 37.8968) (layer "F.SilkS")
     (effects (font (size 0.8 0.8) (thickness 0.1)))
   )
